File: relay-driver-shield.kicad_pcb (KiCad board)
At the start: 2 copper layers, 21 parts, among them J1 Screw_Terminal_01x02, J2 Screw_Terminal_01x02, J3 Screw_Terminal_01x02, J4 Screw_Terminal_01x02, Q1 2N7002, Q2 2N7002, Q3 2N7002, Q4 2N7002

Commit message: Added copper fill to bottom
Connections:
- ARD1 pad GND2: (no net) -> GND
- ARD1 pad GND3: (no net) -> GND
- ARD1 pad GND4: (no net) -> GND
Routing:
- net (no net): track 1.17 -> 0.11 mm
- added copper zone on B.Cu, net GND
Changed lines of the file:
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@@
 (kicad_pcb (version 4) (host pcbnew 4.0.7)
   (general
-    (links 36)
+    (links 39)
     (no_connects 0)
-    (area 102.494999 58.869 178.175001 114.85)
+    (area 0 0 0 0)
     (thickness 1.6)
     (drawings 0)
-    (tracks 79)
+    (tracks 77)
     (zones 0)
     (modules 21)
@@
   (page A4)
   (layers
-    (0 F.Cu signal)
+    (0 F.Cu signal hide)
     (31 B.Cu signal)
-    (33 F.Adhes user)
-    (35 F.Paste user)
+    (33 F.Adhes user hide)
+    (35 F.Paste user hide)
     (37 F.SilkS user)
-    (39 F.Mask user)
-    (40 Dwgs.User user)
-    (41 Cmts.User user)
-    (42 Eco1.User user)
-    (43 Eco2.User user)
-    (44 Edge.Cuts user)
-    (45 Margin user)
-    (47 F.CrtYd user)
-    (49 F.Fab user)
+    (39 F.Mask user hide)
+    (40 Dwgs.User user hide)
+    (41 Cmts.User user hide)
+    (42 Eco1.User user hide)
+    (43 Eco2.User user hide)
+    (44 Edge.Cuts user hide)
+    (45 Margin user hide)
+    (47 F.CrtYd user hide)
+    (49 F.Fab user hide)
   )
   (setup
-    (last_trace_width 0.25)
+    (last_trace_width 1)
     (user_trace_width 0.5)
     (user_trace_width 1)
@@
     (pad_to_mask_clearance 0.2)
     (aux_axis_origin 0 0)
-    (visible_elements FFFFFFFF)
+    (visible_elements FFFF4421)
     (pcbplotparams
       (layerselection 0x00030_80000001)
@@
     (add_net "Net-(Q4-Pad1)")
   )
+  (module Resistors_THT:R_Axial_DIN0207_L6.3mm_D2.5mm_P7.62mm_Horizontal (layer F.Cu)
+    (at 144.78 83.82 45)
+    (descr "Resistor, Axial_DIN0207 series, Axial, Horizontal, pin pitch=7.62mm, 0.25W = 1/4W, length*diameter=6.3*2.5mm^2, http://cdn-reichelt.de/documents/datenblatt/B400/1_4W%23YAG.pdf")
+    (tags "Resistor Axial_DIN0207 series Axial Horizontal pin pitch 7.62mm 0.25W = 1/4W length 6.3mm diameter 2.5mm")
+    (fp_text reference R3 (at 3.81 -2.31 45) (layer F.SilkS)
+      (effects (font (size 1 1) (thickness 0.15)))
+    )
+    (fp_text value 1K (at 3.81 2.31 45) (layer F.Fab)
+      (effects (font (size 1 1) (thickness 0.15)))
+    )
+    (fp_line (start 0.66 -1.25) (end 0.66 1.25) (layer F.Fab) (width 0.1))
+    (fp_line (start 0.66 1.25) (end 6.96 1.25) (layer F.Fab) (width 0.1))
+    (fp_line (start 6.96 1.25) (end 6.96 -1.25) (layer F.Fab) (width 0.1))
+    (fp_line (start 6.96 -1.25) (end 0.66 -1.25) (layer F.Fab) (width 0.1))
+    (fp_line (start 0 0) (end 0.66 0) (layer F.Fab) (width 0.1))
+    (fp_line (start 7.62 0) (end 6.96 0) (layer F.Fab) (width 0.1))
+    (fp_line (start 0.6 -0.98) (end 0.6 -1.31) (layer F.SilkS) (width 0.12))
+    (fp_line (start 0.6 -1.31) (end 7.02 -1.31) (layer F.SilkS) (width 0.12))
+    (fp_line (start 7.02 -1.31) (end 7.02 -0.98) (layer F.SilkS) (width 0.12))
+    (fp_line (start 0.6 0.98) (end 0.6 1.31) (layer F.SilkS) (width 0.12))
+    (fp_line (start 0.6 1.31) (end 7.02 1.31) (layer F.SilkS) (width 0.12))
+    (fp_line (start 7.02 1.31) (end 7.02 0.98) (layer F.SilkS) (width 0.12))
+    (fp_line (start -1.05 -1.6) (end -1.05 1.6) (layer F.CrtYd) (width 0.05))
+    (fp_line (start -1.05 1.6) (end 8.7 1.6) (layer F.CrtYd) (width 0.05))
+    (fp_line (start 8.7 1.6) (end 8.7 -1.6) (layer F.CrtYd) (width 0.05))
+    (fp_line (start 8.7 -1.6) (end -1.05 -1.6) (layer F.CrtYd) (width 0.05))
+    (pad 1 thru_hole circle (at 0 0 45) (size 1.6 1.6) (drill 0.8) (layers *.Cu *.Mask)
+      (net 12 "Net-(Q2-Pad1)"))
+    (pad 2 thru_hole oval (at 7.62 0 45) (size 1.6 1.6) (drill 0.8) (layers *.Cu *.Mask)
+      (net 5 "Net-(ARD1-PadD7)"))
+    (model ${KISYS3DMOD}/Resistors_THT.3dshapes/R_Axial_DIN0207_L6.3mm_D2.5mm_P7.62mm_Horizontal.wrl
+      (at (xyz 0 0 0))
+      (scale (xyz 0.393701 0.393701 0.393701))
+      (rotate (xyz 0 0 0))
+    )
+  )
   (module Arduino:Arduino_Uno_Shield (layer F.Cu)
     (at 109.22 114.3)
@@
     (fp_line (start 0 -53.34) (end 64.516 -53.34) (layer F.SilkS) (width 0.15))
     (pad RST2 thru_hole oval (at 63.627 -25.4) (size 1.7272 1.7272) (drill 1.016) (layers *.Cu *.Mask))
-    (pad GND4 thru_hole oval (at 66.167 -25.4) (size 1.7272 1.7272) (drill 1.016) (layers *.Cu *.Mask))
+    (pad GND4 thru_hole oval (at 66.167 -25.4) (size 1.7272 1.7272) (drill 1.016) (layers *.Cu *.Mask)
+      (net 2 GND))
     (pad MOSI thru_hole oval (at 66.167 -27.94) (size 1.7272 1.7272) (drill 1.016) (layers *.Cu *.Mask))
     (pad SCK thru_hole oval (at 63.627 -27.94) (size 1.7272 1.7272) (drill 1.016) (layers *.Cu *.Mask))
@@
     (pad VIN thru_hole oval (at 45.72 -2.54) (size 1.7272 1.7272) (drill 1.016) (layers *.Cu *.Mask)
       (net 1 +12V))
-    (pad GND3 thru_hole oval (at 43.18 -2.54) (size 1.7272 1.7272) (drill 1.016) (layers *.Cu *.Mask))
-    (pad GND2 thru_hole oval (at 40.64 -2.54) (size 1.7272 1.7272) (drill 1.016) (layers *.Cu *.Mask))
+    (pad GND3 thru_hole oval (at 43.18 -2.54) (size 1.7272 1.7272) (drill 1.016) (layers *.Cu *.Mask)
+      (net 2 GND))
+    (pad GND2 thru_hole oval (at 40.64 -2.54) (size 1.7272 1.7272) (drill 1.016) (layers *.Cu *.Mask)
+      (net 2 GND))
     (pad 5V1 thru_hole oval (at 38.1 -2.54) (size 1.7272 1.7272) (drill 1.016) (layers *.Cu *.Mask))
     (pad 3.3V thru_hole oval (at 35.56 -2.54) (size 1.7272 1.7272) (drill 1.016) (layers *.Cu *.Mask))
@@
   )
   (module Resistors_THT:R_Axial_DIN0207_L6.3mm_D2.5mm_P7.62mm_Horizontal (layer F.Cu)
-    (at 144.78 83.82 45)
-    (descr "Resistor, Axial_DIN0207 series, Axial, Horizontal, pin pitch=7.62mm, 0.25W = 1/4W, length*diameter=6.3*2.5mm^2, http://cdn-reichelt.de/documents/datenblatt/B400/1_4W%23YAG.pdf")
-    (tags "Resistor Axial_DIN0207 series Axial Horizontal pin pitch 7.62mm 0.25W = 1/4W length 6.3mm diameter 2.5mm")
-    (fp_text reference R3 (at 3.81 -2.31 45) (layer F.SilkS)
-      (effects (font (size 1 1) (thickness 0.15)))
-    )
-    (fp_text value 1K (at 3.81 2.31 45) (layer F.Fab)
-      (effects (font (size 1 1) (thickness 0.15)))
-    )
-    (fp_line (start 0.66 -1.25) (end 0.66 1.25) (layer F.Fab) (width 0.1))
-    (fp_line (start 0.66 1.25) (end 6.96 1.25) (layer F.Fab) (width 0.1))
-    (fp_line (start 6.96 1.25) (end 6.96 -1.25) (layer F.Fab) (width 0.1))
-    (fp_line (start 6.96 -1.25) (end 0.66 -1.25) (layer F.Fab) (width 0.1))
-    (fp_line (start 0 0) (end 0.66 0) (layer F.Fab) (width 0.1))
-    (fp_line (start 7.62 0) (end 6.96 0) (layer F.Fab) (width 0.1))
-    (fp_line (start 0.6 -0.98) (end 0.6 -1.31) (layer F.SilkS) (width 0.12))
-    (fp_line (start 0.6 -1.31) (end 7.02 -1.31) (layer F.SilkS) (width 0.12))
-    (fp_line (start 7.02 -1.31) (end 7.02 -0.98) (layer F.SilkS) (width 0.12))
-    (fp_line (start 0.6 0.98) (end 0.6 1.31) (layer F.SilkS) (width 0.12))
-    (fp_line (start 0.6 1.31) (end 7.02 1.31) (layer F.SilkS) (width 0.12))
-    (fp_line (start 7.02 1.31) (end 7.02 0.98) (layer F.SilkS) (width 0.12))
-    (fp_line (start -1.05 -1.6) (end -1.05 1.6) (layer F.CrtYd) (width 0.05))
-    (fp_line (start -1.05 1.6) (end 8.7 1.6) (layer F.CrtYd) (width 0.05))
-    (fp_line (start 8.7 1.6) (end 8.7 -1.6) (layer F.CrtYd) (width 0.05))
-    (fp_line (start 8.7 -1.6) (end -1.05 -1.6) (layer F.CrtYd) (width 0.05))
-    (pad 1 thru_hole circle (at 0 0 45) (size 1.6 1.6) (drill 0.8) (layers *.Cu *.Mask)
-      (net 12 "Net-(Q2-Pad1)"))
-    (pad 2 thru_hole oval (at 7.62 0 45) (size 1.6 1.6) (drill 0.8) (layers *.Cu *.Mask)
-      (net 5 "Net-(ARD1-PadD7)"))
-    (model ${KISYS3DMOD}/Resistors_THT.3dshapes/R_Axial_DIN0207_L6.3mm_D2.5mm_P7.62mm_Horizontal.wrl
-      (at (xyz 0 0 0))
-      (scale (xyz 0.393701 0.393701 0.393701))
-      (rotate (xyz 0 0 0))
-    )
-  )
-  (module Resistors_THT:R_Axial_DIN0207_L6.3mm_D2.5mm_P7.62mm_Horizontal (layer F.Cu)
     (at 143.51 78.105 180)
     (descr "Resistor, Axial_DIN0207 series, Axial, Horizontal, pin pitch=7.62mm, 0.25W = 1/4W, length*diameter=6.3*2.5mm^2, http://cdn-reichelt.de/documents/datenblatt/B400/1_4W%23YAG.pdf")
@@
   )
   (segment (start 124.46 104.14) (end 124.38 104.06) (width 0.25) (layer B.Cu) (net 0) (status 30))
-  (segment (start 147.936308 78.74) (end 147.628154 78.431846) (width 0.25) (layer B.Cu) (net 0) (status 30))
-  (segment (start 147.628154 68.271846) (end 147.011846 68.271846) (width 0.25) (layer B.Cu) (net 0) (status 30))
   (segment (start 115.57 100.33) (end 111.76 100.33) (width 1) (layer B.Cu) (net 1))
   (segment (start 115.57 90.17) (end 111.76 90.17) (width 1) (layer B.Cu) (net 1))
@@
   (segment (start 138.43 102.87) (end 143.51 102.87) (width 1) (layer B.Cu) (net 14))
   (segment (start 143.51 102.87) (end 144.78 104.14) (width 1) (layer B.Cu) (net 14))
+  (zone (net 2) (net_name GND) (layer B.Cu) (hatch edge 0.508)
+    (connect_pads thru_hole_only (clearance 0.508))
+    (min_thickness 0.254)
+    (fill yes (arc_segments 16) (thermal_gap 0.508) (thermal_bridge_width 0.508))
+    (polygon
+      (pts
+        (xy 175.26 62.23) (xy 175.26 73.66) (xy 177.8 76.2) (xy 177.8 110.49) (xy 175.26 113.03)
+        (xy 175.26 114.3) (xy 109.22 114.3) (xy 109.22 60.96) (xy 173.99 60.96)
+      )
+    )
+  )
 )
